File: H1DR21/Design/H1DR21.sch (EAGLE design)
At the start: 26 parts, among them P2 HEXABIT_17.32_NO_P6, U2 TCAN334DCNT, X1 XTALL_CSTCE8M00G52

Commit message: - Changed MCU to G0 - New schematic design - New Layout - Generated documentation - Generated BOM - Deleted old output files (drills, gerber, pick and place)
Parts:
- removed B, C, D: PAD1, Hexabitz:PAD1
- removed C2: 1.00uF, Hexabitz:C-0805-POL
- removed C7, C8, C9: 100nF, Hexabitz:C-0603
- added D2: YELLOW, HEXABITZ_USER_INTERFACE_PARTS:VLMS1300-GS08
- added D3: ORANGE, HEXABITZ_USER_INTERFACE_PARTS:VLMS1300-GS08
- added D5: BOURNS_CDSOD323-T03SCBOURNS_CDSOD323-T03SC_0_0, HEXABITZ_RCLS:BOURNS_CDSOD323-T03SCBOURNS_CDSOD323-T03SC_0_0
- added R8, R9: 270.0R, HEXABITZ_RCLS:R-0603
- added SWD: (no value), pinhead:PINHD-1X3
- C1: value 100nF -> 1uF; device Hexabitz:C-0603 -> HEXABITZ_RCLS:C-0805; CAPACITANCE 100nF -> (none); MFN KEMET -> (none); MPN C0603C104K8RACTU -> (none); OCTOPART_URL https://octopart.com/c0603c104k8ractu-kemet-145075?r=sp&s=9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 -> (none); TOLERANCE 10% -> (none); VOLTAGE_RATING 10V -> (none)
- C3: value 4.7uF -> 100nF; device Hexabitz:C-0805-POL -> HEXABITZ_RCLS:C-0603; CAPACITANCE 4.7uF -> (none); MFN Murata -> (none); MPN GRM21BC81E475KA12L -> (none); OCTOPART_URL https://octopart.com/grm21bc81e475ka12l-murata-10331911?r=s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 -> (none); TOLERANCE 10% -> (none); VOLTAGE_RATING 25V -> (none)
- C4: device Hexabitz:C-0805-POL -> HEXABITZ_RCLS:C-0805; CAPACITANCE 4.7uF -> (none); MFN Murata -> (none); MPN GRM21BC81E475KA12L -> (none); OCTOPART_URL https://octopart.com/grm21bc81e475ka12l-murata-10331911?r=s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 -> (none); TOLERANCE 10% -> (none); VOLTAGE_RATING 25V -> (none)
- C5: value 10nF -> 100nF; device Hexabitz:C-0603 -> HEXABITZ_RCLS:C-0603; CAPACITANCE 10nF -> (none); MFN KEMET -> (none); MPN C0603C103K5RACTU -> (none); OCTOPART_URL https://octopart.com/c0603c103k5ractu-kemet-133094?r=sp&s=R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 -> (none); TOLERANCE 10% -> (none); VOLTAGE_RATING 50V -> (none)
- C6: device Hexabitz:C-0603 -> HEXABITZ_RCLS:C-0603; CAPACITANCE 100nF -> (none); MFN KEMET -> (none); MPN C0603C104K8RACTU -> (none); OCTOPART_URL https://octopart.com/c0603c104k8ractu-kemet-145075?r=sp&s=9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 -> (none); TOLERANCE 10% -> (none); VOLTAGE_RATING 10V -> (none)
- D1: value VLMS1300-GS08 -> RED; device Hexabitz:VLMS1300-GS08 -> HEXABITZ_USER_INTERFACE_PARTS:VLMS1300-GS08
- FB1: device Hexabitz:FB-TDK_MMZ1608Y300B -> HEXABITZ_RCLS:FB-0603
- P2: device Hexabitz:HEXABIT_17.32_NO_P6 -> hexabitz_connectors:HEXABIT_17.32_NO_P6
- R: value PAD1 -> R; device Hexabitz:PAD1 -> HEXABITZ_USER_INTERFACE_PARTS:PINHD-1X1
- R1: value 270.0R -> 0.0R; device Hexabitz:R-0603 -> HEXABITZ_RCLS:R-0603; MPN RC0603FR-07270RL -> RC0603JR-070RL; OCTOPART_URL https://octopart.com/search?q=RC0603FR-07270RL&start=0 -> https://octopart.com/rc0603jr-070rl-yageo-1241539?r=sp&s=X2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; RESISTANCE 270.0 Ohm -> 0.0 Ohm; TOLERANCE 1% -> (none)
- R2: value 10.0K -> 270R; device Hexabitz:R-0603 -> HEXABITZ_RCLS:R-0603; MFN Yageo -> (none); MPN RC0603JR-0710KL -> (none); OCTOPART_URL https://octopart.com/search?q=RC0603JR-0710KL&start=0 -> (none); RESISTANCE 10.0K Ohm -> (none); TOLERANCE 5% -> (none)
- R3: value 0.0R -> 10K; device Hexabitz:R-0603 -> HEXABITZ_RCLS:R-0603; MFN Yageo -> (none); MPN RC0603JR-070RL -> (none); OCTOPART_URL https://octopart.com/rc0603jr-070rl-yageo-1241539?r=sp&s=X2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 -> (none); RESISTANCE 0.0 Ohm -> (none)
- U1: value (none) -> STM32G0B1CEU6QFN_B1CEU6_STM-L; device Hexabitz:STM32F091CBU6 -> HEXABITZ_ICs:STM32G0B1CEU6QFN_B1CEU6_STM-L; SPICEPREFIX (none) -> X
- X1: device Hexabitz:XTALL_CSTCE8M00G52 -> HEXABITZ_RCLS:XTALL_CSTCE8M00G52
Connections:
- removed net B: B.P$1, R2.2, U1.PF11-OSC_BOOT0
- removed net N$10: D1.A, R1.1
- removed net N$14: U1.PF0-OSC_IN, X1.1
- removed net N$15: U1.PF1-OSC_OUT, X1.3
- removed net N$8: R1.2, U1.PA11
- removed net R: C1.1, R.P$1, U1.NRST
- new net CLK: R3.2, SWD.1, SWD.2, U1.PA14-BOOT0
- new net DATA: SWD.3, U1.PA13
- new net N$11: R9.2, U1.PB4
- new net N$3: R2.1, U1.PA6
- new net N$4: C3.1, R.1, U1.PF2-NRST
- new net N$5: U1.PF1-OSC_OUT, X1.1
- new net N$6: U1.PF0-OSC_IN, X1.3
- new net N$7: D2.A, R8.1
- new net N$9: R8.2, U1.PB5
- net CAN_SHDN: now also U1.PA4; no longer U1.PB12
- net CAN_STB: now also U1.PB7; no longer U1.PB15
- net GND: now also C3.2, D2.C, D3.C, D5.A, R1.1, U1.VSS; no longer C1.2, C3.-, C4.-, C6.2, C7.2, C8.2, C9.2, R2.1, U1.EP, U1.VSS_0, U1.VSS_1, U1.VSS_2
- net N$1: now also D1.A, R2.2; no longer D.P$1, U1.PA13
- net N$2: now also D3.A, R9.1; no longer C.P$1, U1.PA14
- net USART1_RX: now also U2.RXD; no longer P2.SD5
- net USART1_TX: now also U2.TXD; no longer P2.SU5
- net USART2_RX: now also P2.SD3; no longer P2.SD2
- net USART2_TX: now also P2.SU3; no longer P2.SU2
- net USART3_RX: now also P2.SD5; no longer P2.SD4
- net USART3_TX: now also P2.SU5; no longer P2.SU4
- net USART4_RX: now also P2.SD2; no longer P2.SD1
- net USART4_TX: now also P2.SU2; no longer P2.SU1
- net USART5_RX: now also P2.SD4, U1.PB1; no longer U1.PB4, U2.RXD
- net USART5_TX: now also P2.SU4, U1.PB0; no longer U1.PB3, U2.TXD
- net USART6_RX: now also P2.SD1, U1.PB9; no longer P2.SD3, U1.PA5
- net USART6_TX: now also P2.SU1, U1.PB8; no longer P2.SU3, U1.PA4
- net VDD: now also D5.C, P2.VDD1, P2.VDD2, P2.VDD3, P2.VDD4, P2.VDD5, P2.VDD6; no longer C3.+, C4.+, C6.1, C7.1, C8.1, C9.1, P2.VCC1, P2.VCC2, P2.VCC3, P2.VCC4, P2.VCC5, P2.VCC6, U1.VBAT, U1.VDDIO2, U1.VDD_0, U1.VDD_1
- net VDDA: now also C1.1, C4.1, C6.1, U1.VBAT, U1.VDD/VDDA, U1.VREF+; no longer C2.+, U1.VDDA
- net VSSA: now also C1.2, C4.2, C6.2, R1.2, U1.VSS/VSSA; no longer C2.-, R3.2, U1.VSS_A
Other:
- note added: "BOOT"
- note added: "H1DR2"
- note added: "H1DR21_Backend￼"
- note added: "H1DR21_Frontend"
- note added: "VDD\VDDA Coupling"
- note added: "Vref Coupling"
- note removed: "0"
- note removed: "H1DR20"
- note removed: "H1DR20_Backend￼"
- note removed: "H1DR20_Frontend"
- note removed: "VBAT"
- note removed: "VDD Coupling"
- note removed: "VDDA Coupling"
- note removed: "VDDIO2 Coupling"
- moved on the sheet: C1, C10, C5, C6, D1, FB1, P1, R1, R2, R3, R4, R5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
